File: docs/10_architecture/master_schematic/STM32.kicad_sch (KiCad schematic)
At the start: 0 parts

Commit message: updated master schematics
Other:
- added sheet States (states.kicad_sch)
Changed lines of the file:
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@@
 	(generator_version "10.0")
 	(paper "A4")
+	(sheet
+		(at 116.84 91.44)
+		(size 15.24 6.35)
+		(exclude_from_sim no)
+		(in_bom yes)
+		(on_board yes)
+		(dnp no)
+		(fields_autoplaced yes)
+		(stroke
+			(width 0.1524)
+			(type solid)
+		)
+		(fill
+			(color 0 0 0 0)
+		)
+		(property "Sheetname" "States"
+			(at 116.84 90.7284 0)
+			(show_name no)
+			(do_not_autoplace no)
+			(effects
+				(font
+					(size 1.27 1.27)
+				)
+				(justify left bottom)
+			)
+		)
+		(property "Sheetfile" "states.kicad_sch"
+			(at 116.84 98.3746 0)
+			(show_name no)
+			(do_not_autoplace no)
+			(effects
+				(font
+					(size 1.27 1.27)
+				)
+				(justify left top)
+			)
+		)
+		(instances
+			(project "master_schematic"
+				(path "/161501ba-58a2-4e54-b00f-2c454c29b444/7e33f781-3aae-4aa0-9862-70bc5b76b4e4"
+					(page "5")
+				)
+			)
+		)
+	)
 )
