File: docs/10_architecture/hardware/sensor_bus_interface/master_sense_buses/master_sense_buses.kicad_pcb (KiCad board)
At the start: 2 copper layers, 74 parts, among them U1 ADS131M04IPWR, U2 ADS131M04IPWR, U3 ACS772LCB-050B-PFF-T, U4 AMC1311BDWVR, U5 AMC1311BDWVR, U6 AMC1311BDWVR, U7 AMC1311BDWVR, U8 AMC1302DWV, U9 OPA330xxD, Y1 CB3LV-3I-8M192000

Commit message: updated PCB Rev1.0
Parts:
- added REF Phase: PinHeader_1x01_P2.54mm_Vertical, Connector_PinHeader_2.54mm:PinHeader_1x01_P2.54mm_Vertical, F.Cu at (154.6, 60.0)
- added REF**: PinHeader_1x01_P2.54mm_Vertical, Connector_PinHeader_2.54mm:PinHeader_1x01_P2.54mm_Vertical, F.Cu at (130.4, 157.6)
- added REF**: PinHeader_1x08_P2.54mm_Vertical, Connector_PinHeader_2.54mm:PinHeader_1x08_P2.54mm_Vertical, F.Cu at (156.4, 112.8)
- added REF**: PinHeader_1x01_P2.54mm_Vertical, Connector_PinHeader_2.54mm:PinHeader_1x01_P2.54mm_Vertical, F.Cu at (126.8, 157.6)
- added REF**: PinHeader_1x01_P2.54mm_Vertical, Connector_PinHeader_2.54mm:PinHeader_1x01_P2.54mm_Vertical, F.Cu at (158.2, 60.0)
- moved R15 80.2 mm to (129.1, 45.6), turned to -90 degrees
- moved R40 79.1 mm to (128.6, 154.3), turned to 0 degrees
- moved C20 72.7 mm to (128.6, 149.6), turned to 0 degrees
- moved U8 65.5 mm to (128.7, 144.3), turned to 90 degrees
- moved U3 60.3 mm to (145.1, 143.0), turned to 180 degrees
- moved C19 58.5 mm to (128.7, 139.0), turned to 0 degrees
- moved R17 56.5 mm to (137.9, 60.8), turned to 90 degrees
- moved R16 56.1 mm to (146.5, 60.8), turned to 90 degrees
- moved R4 55.4 mm to (128.0, 136.3), turned to 90 degrees
- moved R32 54.5 mm to (154.6, 63.5), turned to -90 degrees
- moved R5 54.5 mm to (129.6, 136.3), turned to 90 degrees
- moved R21 52.1 mm to (129.1, 66.5), turned to 90 degrees
- moved C10 51.8 mm to (128.8, 133.9), turned to 180 degrees
- moved R24 48.7 mm to (137.9, 66.5), turned to 90 degrees
- moved R18 48.1 mm to (146.5, 66.5), turned to 90 degrees
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Connections:
- C16 pad 1: Net-(U5-VDD2) -> +3.3V
- U5 pad 8: Net-(U5-VDD2) -> +3.3V
- U8 pad 5: unconnected-(U8-GND2-Pad5) -> GND
Routing:
- net +3.3V: track 0.00 -> 160.7 mm, vias 0 -> 14
- net Net-(U4-GND1): track 0.00 -> 89.4 mm, vias 0 -> 3
- net GNDREF: track 0.00 -> 35.4 mm, vias 0 -> 1
- net 0.6 VDC RAIL: track 0.00 -> 26.3 mm, vias 0 -> 3
- net Net-(U2-AIN0P): track 0.00 -> 19.0 mm
- net Net-(U2-AIN0N): track 0.00 -> 17.4 mm
- net Net-(U1-AIN3N): track 0.00 -> 14.9 mm
- net Net-(U1-AIN0P): track 0.00 -> 14.5 mm
- net Net-(U1-AIN0N): track 0.00 -> 14.2 mm
- net Net-(U1-AIN3P): track 0.00 -> 12.4 mm, vias 0 -> 2
- net +5V: track 0.00 -> 11.7 mm
- net Net-(R30-Pad2): track 0.00 -> 10.5 mm
- net Net-(U1-AIN1P): track 0.00 -> 8.10 mm
- net Net-(R20-Pad1): track 0.00 -> 7.64 mm
- net Net-(R23-Pad1): track 0.00 -> 7.59 mm
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- added copper zone on B.Cu, net GND
Other:
- board outline added: 40 x 118.4 mm
- board text added: "3.3V"
- board text added: "5V"
- board text added: "CS1"
- board text added: "CS2"
- board text added: "GND"
- board text added: "MISO"
- board text added: "MOSI"
- board text added: "RESET"
