File: docs/10_architecture/hardware/sensor_bus_interface/master_sense_buses/master_sense_buses.kicad_sch (KiCad schematic)
At the start: 0 parts

Commit message: created unified schematic for sensing
Parts:
- added C1, C11: .1uF, symbol Device:C
- added C10, C14, C6, C7, C8, C9: 10nF, symbol Device:C
- added C12, C13: 1nF, symbol Device:C
- added C15, C16, C17, C18, C19, C20, C21, C22, C23, C24, C25: 100nF, symbol Device:C
- added C2, C3: 1uF, symbol Device:C
- added C4, C5: 220nF, symbol Device:C
- added R1: 3.1k, SparkFun-Resistor:R_0603_1608Metric, symbol SparkFun-Resistor:R
- added R10, R11, R12, R13, R27, R28, R29, R33, R4, R5, R6, R7, R8, R9: 10Ω, SparkFun-Resistor:R_0603_1608Metric, symbol SparkFun-Resistor:R
- added R14: 1kΩ, SparkFun-Resistor:R_0603_1608Metric, symbol SparkFun-Resistor:R
- added R15, R16: 100k, symbol Device:R_45deg
- added R17: 100k, symbol Device:R
- added R18, R19, R20, R21, R22, R23, R24, R25, R26, R30, R31, R32: 330k, SparkFun-Resistor:R_0603_1608Metric, symbol SparkFun-Resistor:R
- added R2: 6.2k, SparkFun-Resistor:R_0603_1608Metric, symbol SparkFun-Resistor:R
- added R3, R35: 10k, SparkFun-Resistor:R_0603_1608Metric, symbol SparkFun-Resistor:R
- added R34: 45k, SparkFun-Resistor:R_0603_1608Metric, symbol SparkFun-Resistor:R
- added R36, R37, R39: 2kΩ, SparkFun-Resistor:R_0603_1608Metric, symbol SparkFun-Resistor:R
- added R38: 2.94kΩ (E96), SparkFun-Resistor:R_0603_1608Metric, symbol SparkFun-Resistor:R
- added R40: L4CL1206LR100DNR, L4CL1206LR100DNR, symbol L4CL1206LR100DNR:L4CL1206LR100DNR
- added U1, U2: ADS131M04IPWR, Analog_DAC:PW20_TEX-L, symbol ADC_converter:ADS131M04IPWR
- added U3: ACS772LCB-050B-PFF-T, Current_Sense:XDCR_ACS772LCB-050B-PFF-T, symbol Sensor_Current:ACS772LCB-050B-PFF-T
- added U4, U5, U6, U7: AMC1311BDWVR, yes:SOIC127P1150X280-8N, symbol AMC1311BDWVR:AMC1311BDWVR
- added U8: AMC1302DWV, SOIC8_DMV_TEX, symbol amc1302dwv:AMC1302DWV
- added U9: OPA330xxD, Package_SO:SOIC-8_3.9x4.9mm_P1.27mm, symbol Amplifier_Operational:OPA330xxD
- added Y1: CB3LV-3I-8M192000, Oscillator:OSC_CB3LV-3I-8M192000, symbol CB3LV-3I-8M192000:CB3LV-3I-8M192000
Connections:
- new net: C22.2, C23.2, C24.2, R15.1, R16.2, R17.2, U4.3 (SHTDN), U4.4 (GND1), U5.3 (SHTDN), U5.4 (GND1), U6.3 (SHTDN), U6.4 (GND1)
- new net: R40.3, U8.3 (INN)
- new net: R40.4, U8.2 (INP)
- new net: R3.1, Y1.1 (EOH)
- new net: U1.17 (CLKIN), U2.17 (CLKIN), Y1.3 (OUTPUT)
- new net: R12.1, U4.6 (VOUTN)
- new net: C6.1, R12.2, U1.9 (AIN3N)
- new net: C25.1, R34.1, R35.1, U9.3 (+)
- new net: R30.1, R31.2
- new net: R30.2, R33.1, R38.1
- new net: R29.2, U4.2 (VIN)
- new net: R13.1, U4.7 (VOUTP)
- new net: C6.2, R13.2, U1.10 (AIN3P)
- new net: U1.11 (*SYNC/*RESET), U2.11 (*SYNC/*RESET)
- new net: U1.14 (SCLK), U2.14 (SCLK)
- new net: U1.15 (DOUT), U2.15 (DOUT)
- new net: U1.16 (DIN), U2.16 (DIN)
- new net: C5.2, U1.18 (CAP)
- new net: C9.2, R7.2, U1.3 (AIN0P)
- new net: C9.1, R6.2, U1.4 (AIN0N)
- new net: C8.1, R8.2, U1.5 (AIN1N)
- new net: C8.2, R9.2, U1.6 (AIN1P)
- new net: C7.2, R11.2, U1.7 (AIN2P)
- new net: C7.1, R10.2, U1.8 (AIN2N)
- new net: R21.1, R22.2
- new net: R27.2, U6.2 (VIN)
- new net: R8.1, U6.6 (VOUTN)
- new net: R9.1, U6.7 (VOUTP)
- new net: R23.1, R29.1, R36.1
- new net: R22.1, R23.2
- new net: R19.1, R20.2
- new net: R24.1, R25.2
- new net: R10.1, U5.6 (VOUTN)
- new net: R27.1, R39.1
- new net: R4.1, U8.7 (OUTP)
- new net: C10.2, R4.2, U2.3 (AIN0P)
- new net: R31.1, R32.2
- new net: R5.1, U8.6 (OUTN)
- new net: C10.1, R5.2, U2.4 (AIN0N)
- new net: R11.1, U5.7 (VOUTP)
- new net: R14.2, U3.3 (VIOUT)
- new net: R18.1, R19.2
- new net: R33.2, U7.2 (VIN)
- new net: R6.1, U7.6 (VOUTN)
- new net: R7.1, U7.7 (VOUTP)
- new net: C4.1, U2.18 (CAP)
- new net: C14.1, R14.1, U2.5 (AIN1N)
- new net: R28.2, U5.2 (VIN)
- new net: C16.1, U5.8 (VDD2)
- new net: R26.1, R28.1, R37.1
- new net: R25.1, R26.2
- new net +3.3V: C1.2, C12.1, C13.1, C15.1, C17.1, C18.1, C19.1, C2.2, C20.1, C21.1, C22.1, C23.1, C24.1, C3.2, R3.2, R34.2, U1.1 (AVDD), U1.20 (DVDD), U2.1 (AVDD), U2.20 (DVDD), U4.1 (VDD1), U4.8 (VDD2), U5.1 (VDD1), U6.1 (VDD1), U6.8 (VDD2), U7.1 (VDD1), U7.8 (VDD2), U8.1 (VDD1), U8.8 (VDD2), U9.7 (V+), Y1.4 (VCC)
- new net +5V: C11.2, U3.1 (VCC)
- new net +VDC: U3.4 (IP+)
- new net -VDC: C20.2, U8.4 (GND1)
- new net 0.6 VDC RAIL: R36.2, R37.2, R38.2, R39.2, U9.2 (-), U9.6
- new net GND: C1.1, C11.1, C12.2, C13.2, C14.2, C15.2, C16.2, C17.2, C18.2, C19.2, C2.1, C25.2, C3.1, C4.2, C5.1, R35.2, U1.19 (DGND), U1.2 (AGND), U2.19 (DGND), U2.2 (AGND), U2.6 (AIN1P), U3.2 (GND), U4.5 (GND2), U5.5 (GND2), U6.5 (GND2), U7.5 (GND2), U9.4 (V-), Y1.2 (GND)
- new net GNDREF: C21.2, U7.4 (GND1)
- new net This just goes to load positive: U3.5 (IP-)
- new net VAC: R32.1
- new net ϕA: R16.1, R18.2
- new net ϕB: R17.1, R24.2
- new net ϕC: R15.2, R21.2
Other:
- note added: "= MISO"
- note added: "= MOSI"
- note added: "CS1"
- note added: "CS2"
- note added: "DC Load Return"
- note added: "DC_A"
- note added: "DC_V"
- note added: "DRDY"
- note added: "MISO"
- note added: "MOSI"
- note added: "RECT-"
- note added: "SYNC/RESET"
- note added: "ϕA"
- note added: "ϕB"
- note added: "ϕC"
- note added: "ϕref"
- note added: "ϕref (EU)"
- note added: "ϕref (USA)"

Commit message: added switch for reference phase 115v-230v
Parts:
- added R41: 1.54kΩ, SparkFun-Resistor:R_0603_1608Metric, symbol SparkFun-Resistor:R
- added SW1: SW_115D-230S, symbol Switch:SW_SPDT
Connections:
- net 0.6 VDC RAIL: now also SW1.2 (B); no longer R38.2
- net at R30.2, R33.1, R38.1: now also R41.1
- new net: R41.2, SW1.3 (C)
- new net: R38.2, SW1.1 (A)
Other:
- moved on the sheet: R38
Changed lines of the file:
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@@
 	)
 	(junction
-		(at 229.87 50.8)
+		(at 245.11 123.19)
 		(diameter 0)
 		(color 0 0 0 0)
 	)
 	(junction
-		(at 242.57 81.28)
+		(at 229.87 50.8)
 		(diameter 0)
 		(color 0 0 0 0)
 	)
 	(junction
-		(at 55.88 121.92)
+		(at 242.57 81.28)
 		(diameter 0)
 		(color 0 0 0 0)
 	)
 	(junction
-		(at 250.19 123.19)
+		(at 55.88 121.92)
 		(diameter 0)
 		(color 0 0 0 0)
@@
 	)
 	(junction
+		(at 250.19 123.19)
+		(diameter 0)
+		(color 0 0 0 0)
+	)
+	(junction
 		(at 140.97 130.81)
 		(diameter 0)
@@
 	(wire
 		(pts
+			(xy 245.11 123.19) (xy 250.19 123.19)
+		)
+		(stroke
+			(width 0)
+			(type default)
+		)
+	)
+	(wire
+		(pts
 			(xy 160.02 114.3) (xy 147.32 114.3)
 		)
@@
 	(wire
 		(pts
+			(xy 234.95 151.13) (xy 255.27 151.13)
+		)
+		(stroke
+			(width 0)
+			(type default)
+		)
+	)
+	(wire
+		(pts
 			(xy 140.97 80.01) (xy 140.97 81.28)
 		)
@@
 	(wire
 		(pts
+			(xy 271.78 142.24) (xy 255.27 142.24)
+		)
+		(stroke
+			(width 0)
+			(type default)
+		)
+	)
+	(wire
+		(pts
 			(xy 59.69 46.99) (xy 86.36 46.99)
 		)
@@
 	(wire
 		(pts
-			(xy 271.78 142.24) (xy 255.27 142.24)
-		)
-		(stroke
-			(width 0)
-			(type default)
-		)
-	)
-	(wire
-		(pts
 			(xy 50.8 121.92) (xy 50.8 76.2)
 		)
@@
 	(wire
 		(pts
+			(xy 255.27 142.24) (xy 255.27 151.13)
+		)
+		(stroke
+			(width 0)
+			(type default)
+		)
+	)
+	(wire
+		(pts
 			(xy 59.69 46.99) (xy 59.69 44.45)
 		)
@@
 	(wire
 		(pts
-			(xy 255.27 142.24) (xy 255.27 151.13)
-		)
-		(stroke
-			(width 0)
-			(type default)
-		)
-	)
-	(wire
-		(pts
 			(xy 158.75 58.42) (xy 158.75 31.75)
 		)
@@
 	(wire
 		(pts
-			(xy 237.49 123.19) (xy 250.19 123.19)
+			(xy 237.49 123.19) (xy 245.11 123.19)
 		)
 		(stroke
@@
 	(wire
 		(pts
-			(xy 255.27 151.13) (xy 234.95 151.13)
-		)
-		(stroke
-			(width 0)
-			(type default)
-		)
-	)
-	(wire
-		(pts
 			(xy 161.29 66.04) (xy 161.29 34.29)
 		)
@@
 	(symbol
 		(lib_id "power:VDC")
-		(at 250.19 130.81 180)
+		(at 247.65 140.97 180)
 		(unit 1)
 		(body_style 1)
@@
 		(fields_autoplaced yes)
 		(property "Reference" "#PWR050"
-			(at 250.19 127 0)
+			(at 247.65 137.16 0)
 			(hide yes)
 			(show_name no)
@@
 		)
 		(property "Value" "0.6 VDC RAIL"
-			(at 250.19 135.89 0)
+			(at 247.65 146.05 0)
 			(show_name no)
 			(do_not_autoplace no)
@@
 		)
 		(property "Footprint" ""
-			(at 250.19 130.81 0)
+			(at 247.65 140.97 0)
 			(hide yes)
 			(show_name no)
@@
 		)
 		(property "Datasheet" ""
-			(at 250.19 130.81 0)
+			(at 247.65 140.97 0)
 			(hide yes)
 			(show_name no)
@@
 		)
 		(property "Description" "Power symbol creates a global label with name \"VDC\""
-			(at 250.19 130.81 0)
+			(at 247.65 140.97 0)
 			(hide yes)
 			(show_name no)
@@
 	(symbol
 		(lib_id "SparkFun-Resistor:R")
+		(at 250.19 127 90)
+		(unit 1)
+		(body_style 1)
+		(exclude_from_sim no)
+		(in_bom yes)
+		(on_board yes)
+		(in_pos_files yes)
+		(dnp no)
+		(property "Reference" "R41"
+			(at 252.476 125.984 90)
+			(show_name no)
+			(do_not_autoplace no)
+			(effects
+				(font
+					(size 1.27 1.27)
+				)
+				(justify right)
+			)
+		)
+		(property "Value" "1.54kΩ"
+			(at 252.476 128.524 90)
+			(show_name no)
+			(do_not_autoplace no)
+			(effects
+				(font
+					(size 1.27 1.27)
+				)
+				(justify right)
+			)
+		)
+		(property "Footprint" "SparkFun-Resistor:R_0603_1608Metric"
+			(at 254.762 127 0)
+			(hide yes)
+			(show_name no)
+			(do_not_autoplace no)
+			(effects
+				(font
+					(size 1.27 1.27)
+				)
+			)
+		)
+		(property "Datasheet" "https://www.vishay.com/docs/20035/dcrcwe3.pdf"
+			(at 259.08 128.27 0)
+			(hide yes)
+			(show_name no)
+			(do_not_autoplace no)
+			(effects
+				(font
+					(size 1.27 1.27)
+				)
+			)
+		)
+		(property "Description" "Resistor"
+			(at 261.62 127 0)
+			(hide yes)
+			(show_name no)
+			(do_not_autoplace no)
+			(effects
+				(font
+					(size 1.27 1.27)
+				)
+			)
+		)
+		(property "PROD_ID" "RES-07856"
+			(at 257.048 127 0)
+			(hide yes)
+			(show_name no)
+			(do_not_autoplace no)
+			(effects
+				(font
+					(size 1.27 1.27)
+				)
+			)
+		)
+		(pin "1"
+		)
+		(pin "2"
+		)
+		(instances
+			(project "master_sense_buses"
+				(path "/b64a929e-7a8b-44c9-a2ae-ae2740f738e8"
+					(reference "R41")
+					(unit 1)
+				)
+			)
+		)
+	)
+	(symbol
+		(lib_id "SparkFun-Resistor:R")
 		(at 180.34 66.04 0)
 		(unit 1)
@@
 	(symbol
 		(lib_id "SparkFun-Resistor:R")
-		(at 250.19 127 90)
+		(at 245.11 127 90)
 		(unit 1)
 		(body_style 1)
@@
 		(in_pos_files yes)
 		(dnp no)
-		(fields_autoplaced yes)
 		(property "Reference" "R38"
-			(at 252.73 125.7299 90)
+			(at 238.252 118.11 90)
 			(show_name no)
 			(do_not_autoplace no)
@@
 		)
 		(property "Value" "2.94kΩ (E96)"
-			(at 252.73 128.2699 90)
+			(at 238.252 120.65 90)
 			(show_name no)
 			(do_not_autoplace no)
@@
 		)
 		(property "Footprint" "SparkFun-Resistor:R_0603_1608Metric"
-			(at 254.762 127 0)
+			(at 249.682 127 0)
 			(hide yes)
 			(show_name no)
@@
 		)
 		(property "Datasheet" "https://www.vishay.com/docs/20035/dcrcwe3.pdf"
-			(at 259.08 128.27 0)
+			(at 254 128.27 0)
 			(hide yes)
 			(show_name no)
@@
 		)
 		(property "Description" "Resistor"
-			(at 261.62 127 0)
+			(at 256.54 127 0)
 			(hide yes)
 			(show_name no)
@@
 		)
 		(property "PROD_ID" "RES-07856"
-			(at 257.048 127 0)
+			(at 251.968 127 0)
 			(hide yes)
 			(show_name no)
@@
 					(unit 1)
 				)
+			)
+		)
+	)
+	(symbol
+		(lib_id "Switch:SW_SPDT")
+		(at 247.65 135.89 90)
+		(unit 1)
+		(body_style 1)
+		(exclude_from_sim no)
+		(in_bom yes)
+		(on_board yes)
+		(in_pos_files yes)
+		(dnp no)
+		(fields_autoplaced yes)
+		(property "Reference" "SW1"
+			(at 252.73 134.6199 90)
+			(show_name no)
+			(do_not_autoplace no)
+			(effects
+				(font
+					(size 1.27 1.27)
+				)
+				(justify right)
+			)
+		)
+		(property "Value" "SW_115D-230S"
+			(at 252.73 137.1599 90)
+			(show_name no)
+			(do_not_autoplace no)
+			(effects
+				(font
+					(size 1.27 1.27)
+				)
+				(justify right)
+			)
+		)
+		(property "Footprint" ""
+			(at 247.65 135.89 0)
+			(hide yes)
+			(show_name no)
+			(do_not_autoplace no)
+			(effects
+				(font
+					(size 1.27 1.27)
+				)
+			)
+		)
+		(property "Datasheet" ""
+			(at 255.27 135.89 0)
+			(hide yes)
+			(show_name no)
+			(do_not_autoplace no)
+			(effects
+				(font
+					(size 1.27 1.27)
+				)
+			)
+		)
+		(property "Description" "Switch, single pole double throw"
+			(at 247.65 135.89 0)
+			(hide yes)
+			(show_name no)
+			(do_not_autoplace no)
+			(effects
+				(font
+					(size 1.27 1.27)
+				)
+			)
+		)
+		(pin "3"
+		)
+		(pin "2"
+		)
+		(pin "1"
+		)
+		(instances
+			(project "master_sense_buses"
+				(path "/b64a929e-7a8b-44c9-a2ae-ae2740f738e8"
+					(reference "SW1")
+					(unit 1)
+				)

Commit message: updated schematic/footprints, updated pcb
Parts:
- removed R1: 3.1k, SparkFun-Resistor:R_0603_1608Metric, symbol SparkFun-Resistor:R
- removed R2: 6.2k, SparkFun-Resistor:R_0603_1608Metric, symbol SparkFun-Resistor:R
- removed SW1: SW_115D-230S, symbol Switch:SW_SPDT
- C1, C11, C12, C13, C15, C16, C17, C18, C19, C2, C20, C21, C22, C23, C24, C25, C3, C4, C5: footprint (none) -> Capacitor_SMD:C_0201_0603Metric
- C10, C14, C6, C7, C8, C9: footprint (none) -> Capacitor_SMD:C_0603_1608Metric
- R10, R11, R12, R13, R14, R3, R34, R4, R5, R6, R7, R8, R9: footprint SparkFun-Resistor:R_0603_1608Metric -> Resistor_SMD:R_0603_1608Metric
- R15, R16, R17: footprint (none) -> Resistor_THT:R_Axial_DIN0414_L11.9mm_D4.5mm_P15.24mm_Horizontal
- R18, R19, R20, R21, R22, R23, R24, R25, R26, R30, R31, R32, R36, R37, R38, R39, R41: footprint SparkFun-Resistor:R_0603_1608Metric -> Resistor_SMD:R_1206_3216Metric
- R27, R28, R29, R33: value 10Ω -> 100Ω; footprint SparkFun-Resistor:R_0603_1608Metric -> Resistor_SMD:R_0805_2012Metric
- R35: footprint SparkFun-Resistor:R_0603_1608Metric -> Resistor_SMD:R_0201_0603Metric
- R40: footprint L4CL1206LR100DNR -> yes:L4CL1206LR100DNR
- U8: footprint SOIC8_DMV_TEX -> yes:SOIC8_DMV_TEX-L
Connections:
- net GNDREF: now also U7.3 (SHTDN)
- net at R20.1: now also R27.1, R39.1
Other:
- note removed: "ϕref (EU)"
- note removed: "ϕref (USA)"

Commit message: updated PCB Rev1.0
Connections:
- net +3.3V: now also C16.1, U5.8 (VDD2)
- net GND: now also U8.5 (GND2)
Changed lines of the file:
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@@
 	)
 	(junction
+		(at 194.31 68.58)
+		(diameter 0)
+		(color 0 0 0 0)
+	)
+	(junction
 		(at 50.8 76.2)
 		(diameter 0)
@@
 	(symbol
 		(lib_id "power:GND")
-		(at 194.31 140.97 270)
+		(at 194.31 148.59 180)
 		(unit 1)
 		(body_style 1)
@@
 		(dnp no)
 		(property "Reference" "#PWR013"
-			(at 187.96 140.97 0)
+			(at 194.31 142.24 0)
 			(hide yes)
 			(show_name no)
@@
 		)
 		(property "Value" "GND"
-			(at 189.484 140.97 90)
+			(at 194.31 143.764 90)
 			(show_name no)
 			(do_not_autoplace no)
@@
 		)
 		(property "Footprint" ""
-			(at 194.31 140.97 0)
+			(at 194.31 148.59 0)
 			(hide yes)
 			(show_name no)
@@
 		)
 		(property "Datasheet" ""
-			(at 194.31 140.97 0)
+			(at 194.31 148.59 0)
 			(hide yes)
 			(show_name no)
@@
 		)
 		(property "Description" "Power symbol creates a global label with name \"GND\" , ground"
-			(at 194.31 140.97 0)
+			(at 194.31 148.59 0)
 			(hide yes)
 			(show_name no)
@@
 	(symbol
 		(lib_id "power:+3.3V")
-		(at 194.2043 68.58 90)
+		(at 194.31 68.58 90)
 		(unit 1)
 		(body_style 1)
@@
 		(fields_autoplaced yes)
 		(property "Reference" "#PWR027"
-			(at 198.0143 68.58 0)
+			(at 198.12 68.58 0)
 			(hide yes)
 			(show_name no)
@@
 		)
 		(property "Value" "+3.3V"
-			(at 190.3943 68.5799 90)
+			(at 190.5 68.5799 90)
 			(show_name no)
 			(do_not_autoplace no)
@@
 		)
 		(property "Footprint" ""
-			(at 194.2043 68.58 0)
+			(at 194.31 68.58 0)
 			(hide yes)
 			(show_name no)
@@
 		)
 		(property "Datasheet" ""
-			(at 194.2043 68.58 0)
+			(at 194.31 68.58 0)
 			(hide yes)
 			(show_name no)
@@
 		)
 		(property "Description" "Power symbol creates a global label with name \"+3.3V\""
-			(at 194.2043 68.58 0)
+			(at 194.31 68.58 0)
 			(hide yes)
 			(show_name no)
